File: RookBril.kicad_sch (KiCad schematic)
At the start: 2 parts, among them U2 STM32F411RETx, U3 VNH7070ASTR

Commit message: updated schematic
alles toegevoegd aan de schematic
Parts:
- added C1, C9: 4.7u, symbol Device:C
- added C2, C3, C4, C5, C8: 100n, symbol Device:C
- added C6: 10n, symbol Device:C
- added C7: 1u, symbol Device:C
- added D2: LOW-BAT_LED, symbol Device:LED
- added FB1: FerriteBead, symbol Device:FerriteBead
- added J1: IR_SENSOR0_PINS, symbol Connector:Conn_01x03_Pin
- added J2, J4: IR_SENSOR2_PINS, symbol Connector:Conn_01x03_Pin
- added J3: IR_SENSOR1_PINS, symbol Connector:Conn_01x03_Pin
- added J6: PDLC_JST_PINS, symbol Connector:Conn_01x02_Pin
- added J7: PROGRAM_PINS, symbol Connector_Generic:Conn_02x05_Counter_Clockwise
- added J?: MCU_MODE_PINS, symbol Connector:Conn_01x03_Pin
- added J?: BATT_PINS, symbol Connector:Conn_01x02_Socket
- added R1: 10k, symbol Device:R
- added R13: R, symbol Device:R
- added R2: 50K, symbol Device:R
- added R3: 100K, symbol Device:R
- added SW1: SW_Push, symbol Switch:SW_Push
- renumbered U3 to U1
Connections:
- net +3V0: now reaches U2.1 (VBAT)
- net +3V0: now also U1.13 (CS), U2.19 (VDD), U2.32 (VDD), U2.48 (VDD), U2.64 (VDD), C1.1, C2.1, C3.1, C4.1, C5.1, FB1.1, J1.1 (Pin_1), J2.1 (Pin_1), J3.1 (Pin_1), J4.1 (Pin_1), J7.1 (Pin_1), J?.1 (Pin_1), R1.1
- net GND: now reaches U2.12 (VSSA)
- net GND: now also U1.1 (GND), U1.16 (GND), U1.8 (GND), U1.9 (GND), U2.18 (VSS), U2.31 (VSS), U2.47 (VSS), U2.63 (VSS), C1.2, C2.2, C3.2, C4.2, C5.2, C6.2, C7.2, C8.2, C9.2, D2.1 (K), J1.3 (Pin_3), J2.3 (Pin_3), J3.3 (Pin_3), J4.3 (Pin_3), J7.2 (Pin_2), J7.3 (Pin_3), J7.5 (Pin_5), J?.1 (Pin_1), J?.3 (Pin_3), R3.2, SW1.1
- net VDDA: now reaches U2.13 (VDDA)
- net VDDA: now also C6.1, C7.1, FB1.2
- net IR_SIG0: now reaches U2.14 (PA0)
- net IR_SIG0: now also J1.2 (Pin_2)
- net IR_SIG1: now reaches U2.15 (PA1)
- net IR_SIG1: now also J3.2 (Pin_2)
- net IR_SIG2: now reaches U2.16 (PA2)
- net IR_SIG2: now also J2.2 (Pin_2)
- net IR_SIG3: now reaches U2.17 (PA3)
- net IR_SIG3: now also J4.2 (Pin_2)
- net H-BRIDGE_PWM: now reaches U2.20 (PA4)
- net H-BRIDGE_PWM: now also U1.11 (PWM)
- net H-BRIDGE_SEL: now reaches U2.21 (PA5)
- net H-BRIDGE_SEL: now also U1.14 (SEL_0)
- net H-BRIDGE_IN_A: now reaches U2.22 (PA6)
- net H-BRIDGE_IN_A: now also U1.3 (IN_A)
- net H-BRIDGE_IN_B: now reaches U2.23 (PA7)
- net H-BRIDGE_IN_B: now also U1.6 (IN_B)
- net VBAT_FB: now reaches U2.24 (PC4)
- net VBAT_FB: now also R2.2, R3.1
- net PDLC-BOOST_VOUT-FB: now reaches U2.25 (PC5)
- net PDLC-BOOST_CTRL: now reaches U2.26 (PB0)
- net at U2.27 (PB1): now also R13.1
- net at U2.30 (VCAP1): now also C9.1
- net SWDIO: now reaches U2.46 (PA13)
- net SWDIO: now also J7.10 (Pin_10)
- net SDCLK: now reaches U2.49 (PA14)
- net SDCLK: now also J7.9 (Pin_9)
- net SWO: now reaches U2.55 (PB3)
- net SWO: now also J7.8 (Pin_8)
- net at U2.60 (BOOT0): now also J?.2 (Pin_2)
- net NRST: now reaches U2.7 (NRST)
- net NRST: now also C8.1, J7.6 (Pin_6), R1.2, SW1.2
- net at U1.10 (OUT_B), U1.7 (OUT_B): now also J6.2 (Pin_2)
- net VCC: now reaches U1.12 (VCC), U1.4 (VCC), U1.5 (VCC)
- net at U1.15 (OUT_A), U1.2 (OUT_A): now also J6.1 (Pin_1)
- new net: D2.2 (A), R13.2
- new net +BATT: J?.2 (Pin_2), R2.1
- no-connect marks 0 -> 37
Other:
- sheet Power renamed PDLC boost
- added sheet 3V_BUCK-BOOST (3V_BUCK-BOOST.kicad_sch)
- note added: "0.8-1.5V/cell 3 cell 2.4-4.5V totaal"
- note added: "H-BRIDGE FOR PDLC"
- note added: "PROGRAMMING INTERFACE"
- note added: "VBAT VOLTAGE DIVIDER TO MEASURE"
- moved on the sheet: U1, U2

Commit message: footprint assignments gedaan + verbeteringen
Parts:
- removed C6: 10n, symbol Device:C
- removed C7: 1u, symbol Device:C
- removed C8: 100n, symbol Device:C
- removed C9: 4.7u, symbol Device:C
- removed D2: LOW-BAT_LED, symbol Device:LED
- removed FB1: FerriteBead, symbol Device:FerriteBead
- removed J2: IR_SENSOR2_PINS, symbol Connector:Conn_01x03_Pin
- removed J7: PROGRAM_PINS, symbol Connector_Generic:Conn_02x05_Counter_Clockwise
- removed J?: MCU_MODE_PINS, symbol Connector:Conn_01x03_Pin
- removed SW1: SW_Push, symbol Switch:SW_Push
- removed U2: STM32F411RETx, Package_QFP:LQFP-64_10x10mm_P0.5mm, symbol MCU_ST_STM32F4:STM32F411RETx
- added J5: IR_SENSOR3_PINS, Connector_PinHeader_2.54mm:PinHeader_1x03_P2.54mm_Vertical, symbol Connector:Conn_01x03_Pin
- added J6: LOW-BAT_LED_CONN, Connector_PinHeader_2.54mm:PinHeader_1x02_P2.54mm_Vertical, symbol Connector:Conn_01x02_Pin
- added R2, R5, R6: R, Resistor_SMD:R_0805_2012Metric_Pad1.20x1.40mm_HandSolder, symbol Device:R
- C1: value 4.7u -> 100n; footprint (none) -> Capacitor_SMD:C_0805_2012Metric_Pad1.18x1.45mm_HandSolder; now not fitted
- C2, C3, C4: footprint (none) -> Capacitor_SMD:C_0805_2012Metric_Pad1.18x1.45mm_HandSolder; now not fitted
- C5: footprint (none) -> Capacitor_SMD:C_0805_2012Metric_Pad1.18x1.45mm_HandSolder
- J2: renamed from J1; footprint (none) -> Connector_PinHeader_2.54mm:PinHeader_1x03_P2.54mm_Vertical
- J3, J4: footprint (none) -> Connector_PinHeader_2.54mm:PinHeader_1x03_P2.54mm_Vertical
- J7: renamed from J6; footprint (none) -> Connector_PinHeader_2.54mm:PinHeader_1x02_P2.54mm_Vertical
- J?: footprint (none) -> Connector_PinHeader_2.54mm:PinHeader_1x02_P2.54mm_Vertical
- R1: value 10k -> R; footprint (none) -> Resistor_SMD:R_0805_2012Metric_Pad1.20x1.40mm_HandSolder
- R3: renamed from R2; footprint (none) -> Resistor_SMD:R_0805_2012Metric_Pad1.20x1.40mm_HandSolder
- R4: renamed from R3; footprint (none) -> Resistor_SMD:R_0805_2012Metric_Pad1.20x1.40mm_HandSolder
- R7: renamed from R13; value R -> undetermined; footprint (none) -> Resistor_SMD:R_0805_2012Metric_Pad1.20x1.40mm_HandSolder
Connections:
- net +3V0: now also R2.1, R5.1, R6.1; no longer C5.1, J2.1 (Pin_1), J3.1 (Pin_1), J4.1 (Pin_1)
- net GND: now also J5.3 (Pin_3), J6.1 (Pin_1)
- net IR_SIG2: now also J4.2 (Pin_2)
- net IR_SIG3: now also J5.2 (Pin_2); no longer J4.2 (Pin_2)
- net VCC: now also C5.1
- net MCU/LOW-BAT_LED_EN: now reaches R7.1
- net at R7.2: now also J6.2 (Pin_2)
- net NRST: no longer names the net of R1.2
- net NRST: now also J2.1 (Pin_1)
- new net: J4.1 (Pin_1), R5.2
- new net: J3.1 (Pin_1), R2.2
- new net: J5.1 (Pin_1), R6.2
- no-connect marks 37 -> 0
Other:
- added sheet MCU (MCU.kicad_sch)
- note added: "IR sensors"
- note added: "battery connect"
- note added: "power flags"
- note removed: "PROGRAMMING INTERFACE"
- moved on the sheet: J2, J7, J?, R3, R4, R7, U1

Commit message: aantal componenten veranderd.
Parts:
- added C3: 100n, Capacitor_SMD:C_0805_2012Metric_Pad1.18x1.45mm_HandSolder, symbol Device:C
- renumbered C3 to C4, C4 to C5, C5 to C6
Connections:
- net GND: now also C3.2
- net VBAT_FB: now also C3.1
Changed lines of the file:
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@@
   (junction (at 208.28 59.69) (diameter 0) (color 0 0 0 0)
   )
+  (junction (at 151.13 51.435) (diameter 0) (color 0 0 0 0)
+  )
+  (junction (at 140.97 40.005) (diameter 0) (color 0 0 0 0)
+  )
   (junction (at 151.13 40.005) (diameter 0) (color 0 0 0 0)
   )
@@
     (stroke (width 0) (type default))
   )
+  (wire (pts (xy 140.97 51.435) (xy 151.13 51.435))
+    (stroke (width 0) (type default))
+  )
   (wire (pts (xy 202.565 104.14) (xy 202.565 102.235))
     (stroke (width 0) (type default))
   )
+  (wire (pts (xy 140.97 42.545) (xy 140.97 40.005))
+    (stroke (width 0) (type default))
+  )
   (wire (pts (xy 82.55 89.535) (xy 86.36 89.535))
     (stroke (width 0) (type default))
@@
     (stroke (width 0) (type default))
   )
-  (wire (pts (xy 143.51 40.005) (xy 151.13 40.005))
+  (wire (pts (xy 139.7 40.005) (xy 140.97 40.005))
     (stroke (width 0) (type default))
   )
@@
     (stroke (width 0) (type default))
   )
+  (wire (pts (xy 151.13 51.435) (xy 151.13 50.165))
+    (stroke (width 0) (type default))
+  )
+  (wire (pts (xy 140.97 40.005) (xy 151.13 40.005))
+    (stroke (width 0) (type default))
+  )
+  (wire (pts (xy 140.97 50.165) (xy 140.97 51.435))
+    (stroke (width 0) (type default))
+  )
   (wire (pts (xy 187.96 137.16) (xy 195.58 137.16))
     (stroke (width 0) (type default))
@@
   )
   (wire (pts (xy 151.13 25.4) (xy 151.13 29.845))
+    (stroke (width 0) (type default))
+  )
+  (wire (pts (xy 151.13 52.705) (xy 151.13 51.435))
     (stroke (width 0) (type default))
   )
@@
     (effects (font (size 1.27 1.27)) (justify left bottom))
   )
-  (label "VBAT_FB" (at 143.51 40.005 180) (fields_autoplaced)
+  (label "VBAT_FB" (at 139.7 40.005 180) (fields_autoplaced)
     (effects (font (size 1.27 1.27)) (justify right bottom))
   )
@@
     )
   )
+  (symbol (lib_id "Device:C") (at 140.97 46.355 0) (unit 1)
+    (in_bom yes) (on_board yes) (dnp no) (fields_autoplaced)
+    (property "Reference" "C3" (at 144.145 45.72 0)
+      (effects (font (size 1.27 1.27)) (justify left))
+    )
+    (property "Value" "100n" (at 144.145 48.26 0)
+      (effects (font (size 1.27 1.27)) (justify left))
+    )
+    (property "Footprint" "Capacitor_SMD:C_0805_2012Metric_Pad1.18x1.45mm_HandSolder" (at 141.9352 50.165 0)
+      (effects (font (size 1.27 1.27)) hide)
+    )
+    (property "Datasheet" "~" (at 140.97 46.355 0)
+      (effects (font (size 1.27 1.27)) hide)
+    )
+    (pin "1")
+    (pin "2")
+    (instances
+      (project "RookBril"
+        (path "/5dc439a9-720d-4bdc-b61f-78a76fde4df5"
+          (reference "C3") (unit 1)
+        )
+      )
+    )
+  )
   (symbol (lib_id "power:+3V0") (at 208.28 22.225 0) (unit 1)
     (in_bom yes) (on_board yes) (dnp no) (fields_autoplaced)
@@
   (symbol (lib_id "Device:C") (at 202.565 107.95 0) (unit 1)
     (in_bom yes) (on_board yes) (dnp no) (fields_autoplaced)
-    (property "Reference" "C5" (at 205.74 107.315 0)
+    (property "Reference" "C6" (at 205.74 107.315 0)
       (effects (font (size 1.27 1.27)) (justify left))
     )
@@
       (project "RookBril"
         (path "/5dc439a9-720d-4bdc-b61f-78a76fde4df5"
-          (reference "C5") (unit 1)
+          (reference "C6") (unit 1)
         )
       )
@@
   (symbol (lib_id "Device:C") (at 208.28 66.04 0) (unit 1)
     (in_bom yes) (on_board yes) (dnp yes) (fields_autoplaced)
-    (property "Reference" "C3" (at 211.455 65.405 0)
+    (property "Reference" "C4" (at 211.455 65.405 0)
       (effects (font (size 1.27 1.27)) (justify left))
     )
@@
       (project "RookBril"
         (path "/5dc439a9-720d-4bdc-b61f-78a76fde4df5"
-          (reference "C3") (unit 1)
+          (reference "C4") (unit 1)
         )
       )
@@
   (symbol (lib_id "Device:C") (at 252.73 66.04 0) (unit 1)
     (in_bom yes) (on_board yes) (dnp yes) (fields_autoplaced)
-    (property "Reference" "C4" (at 255.905 65.405 0)
+    (property "Reference" "C5" (at 255.905 65.405 0)
       (effects (font (size 1.27 1.27)) (justify left))
     )
@@
       (project "RookBril"
         (path "/5dc439a9-720d-4bdc-b61f-78a76fde4df5"
-          (reference "C4") (unit 1)
+          (reference "C5") (unit 1)
         )
       )
@@
     )
   )
-  (symbol (lib_id "power:GND") (at 151.13 50.165 0) (unit 1)
-    (in_bom yes) (on_board yes) (dnp no) (fields_autoplaced)
-    (property "Reference" "#PWR015" (at 151.13 56.515 0)
-      (effects (font (size 1.27 1.27)) hide)
-    )
-    (property "Value" "GND" (at 151.13 54.61 0)
-      (effects (font (size 1.27 1.27)))
-    )
-    (property "Footprint" "" (at 151.13 50.165 0)
-      (effects (font (size 1.27 1.27)) hide)
-    )
-    (property "Datasheet" "" (at 151.13 50.165 0)
-      (effects (font (size 1.27 1.27)) hide)
-    )
+  (symbol (lib_id "power:GND") (at 151.13 52.705 0) (unit 1)
+    (in_bom yes) (on_board yes) (dnp no) (fields_autoplaced)
+    (property "Reference" "#PWR015" (at 151.13 59.055 0)
+      (effects (font (size 1.27 1.27)) hide)
+    )
+    (property "Value" "GND" (at 151.13 57.15 0)
+      (effects (font (size 1.27 1.27)))
+    )
+    (property "Footprint" "" (at 151.13 52.705 0)
+      (effects (font (size 1.27 1.27)) hide)
+    )
+    (property "Datasheet" "" (at 151.13 52.705 0)
+      (effects (font (size 1.27 1.27)) hide)
+    )

Commit message: Klein beetje reorganiseren van de lay-out Silkscreen schoongemaakt TestPoints en Mounting holes toegevoegd
Parts:
- added H1, H2, H3, H4: MountingHole, MountingHole:MountingHole_3mm, symbol Mechanical:MountingHole
- added TP1, TP2, TP4: TestPoint, TestPoint:TestPoint_Plated_Hole_D2.0mm, symbol Connector:TestPoint
Connections:
- net +3V0: now also TP1.1
- net GND: now also TP4.1
- net VCC: now also TP2.1

Commit message: updated schematic en interactive bom in de git
Parts:
- added TP3: TestPoint, Components:exposedPad5x10, symbol Connector:TestPoint
Connections:
- net GND: now also TP3.1
Changed lines of the file:
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@@
+    (stroke (width 0) (type default))
+  )
+  (wire (pts (xy 27.94 77.47) (xy 27.94 74.93))
     (stroke (width 0) (type default))
   )
@@
     )
   )
+  (symbol (lib_id "power:GND") (at 27.94 77.47 0) (unit 1)
+    (in_bom yes) (on_board yes) (dnp no) (fields_autoplaced)
+    (property "Reference" "#PWR?" (at 27.94 83.82 0)
+      (effects (font (size 1.27 1.27)) hide)
+    )
+    (property "Value" "GND" (at 27.94 81.28 0)
+      (effects (font (size 1.27 1.27)))
+    )
+    (property "Footprint" "" (at 27.94 77.47 0)
+      (effects (font (size 1.27 1.27)) hide)
+    )
+    (property "Datasheet" "" (at 27.94 77.47 0)
+      (effects (font (size 1.27 1.27)) hide)
+    )
+    (pin "1")
+    (instances
+      (project "RookBril"
+        (path "/5dc439a9-720d-4bdc-b61f-78a76fde4df5/2d26b15a-54d8-4f7d-a410-dc25ffe321a1"
+          (reference "#PWR?") (unit 1)
+        )
+        (path "/5dc439a9-720d-4bdc-b61f-78a76fde4df5"
+          (reference "#PWR056") (unit 1)
+        )
+      )
+    )
+  )
   (symbol (lib_id "Mechanical:MountingHole") (at 87.63 53.34 0) (unit 1)
     (in_bom yes) (on_board yes) (dnp no) (fields_autoplaced)
@@
         )
       )
+    )
+  )
+  (symbol (lib_id "Connector:TestPoint") (at 27.94 74.93 0) (unit 1)
+    (in_bom yes) (on_board yes) (dnp no)
+    (property "Reference" "TP3" (at 26.67 68.58 0)
+      (effects (font (size 1.27 1.27)) (justify left))
+    )
+    (property "Value" "TestPoint" (at 24.13 66.04 0)
+      (effects (font (size 1.27 1.27)) (justify left))
+    )
+    (property "Footprint" "Components:exposedPad5x10" (at 33.02 74.93 0)
+      (effects (font (size 1.27 1.27)) hide)
+    )
+    (property "Datasheet" "~" (at 33.02 74.93 0)
+      (effects (font (size 1.27 1.27)) hide)
+    )
+    (pin "1")
+    (instances
+      (project "RookBril"
+        (path "/5dc439a9-720d-4bdc-b61f-78a76fde4df5"
+          (reference "TP3") (unit 1)
+        )
+      )

Commit message: kleine dingen
Parts:
- R3: value 50K -> 51k
Connections:
- net +3V0: no longer U1.13 (CS)
- no-connect marks 0 -> 2
Changed lines of the file:
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@@
   (junction (at 252.73 28.575) (diameter 0) (color 0 0 0 0)
   )
+  (no_connect (at 210.82 121.92))
+  (no_connect (at 195.58 127))
   (wire (pts (xy 195.58 142.24) (xy 182.245 142.24))
     (stroke (width 0) (type default))
@@
     (stroke (width 0) (type default))
   )
-  (wire (pts (xy 195.58 127) (xy 184.15 127))
-    (stroke (width 0) (type default))
-  )
   (wire (pts (xy 240.03 33.655) (xy 240.03 37.465))
     (stroke (width 0) (type default))
@@
   )
   (wire (pts (xy 248.92 59.69) (xy 252.73 59.69))
-    (stroke (width 0) (type default))
-  )
-  (wire (pts (xy 184.15 118.11) (xy 184.15 127))
     (stroke (width 0) (type default))
   )
@@
       (effects (font (size 1.27 1.27)) (justify left))
     )
-    (property "Value" "50K" (at 153.67 35.56 0)
+    (property "Value" "51k" (at 153.67 35.56 0)
       (effects (font (size 1.27 1.27)) (justify left))
     )
@@
         )
       )
-    )
-  )
-  (symbol (lib_id "power:+3V0") (at 184.15 118.11 0) (unit 1)
-    (in_bom yes) (on_board yes) (dnp no) (fields_autoplaced)
-    (property "Reference" "#PWR025" (at 184.15 121.92 0)
-      (effects (font (size 1.27 1.27)) hide)
-    )
-    (property "Value" "+3V0" (at 184.15 114.3 0)
-      (effects (font (size 1.27 1.27)))
-    )
-    (property "Footprint" "" (at 184.15 118.11 0)
-      (effects (font (size 1.27 1.27)) hide)
-    )
-    (property "Datasheet" "" (at 184.15 118.11 0)
-      (effects (font (size 1.27 1.27)) hide)
-    )
-    (pin "1")
-    (instances
-      (project "RookBril"
-        (path "/5dc439a9-720d-4bdc-b61f-78a76fde4df5"
-          (reference "#PWR025") (unit 1)
-        )
-      )
